Commit message: Update 8DOFROBOT2 joint limits

File: robot_description/8DOFROBOT2/urdf/8DOFROBOT2.urdf (robot description, URDF)
Before this commit: robot 8DOFROBOT2, 9 links, 8 joints
Joints:
- joint left_hip_joint: limit lower=0 upper=0 effort=0 velocity=0 -> lower=-0.9075712110370514 upper=0.9075712110370514 effort=0 velocity=0
- joint left_knee_joint : limit lower=0 upper=0 effort=0 velocity=0 -> lower=-2.792526803190927 upper=0 effort=0 velocity=0
- joint left_thigh_joint: limit lower=0 upper=0 effort=0 velocity=0 -> lower=-0.8726646259971648 upper=1.3089969389957472 effort=0 velocity=0
- joint right_hip_joint: limit lower=0 upper=0 effort=0 velocity=0 -> lower=-0.9075712110370514 upper=0.9075712110370514 effort=0 velocity=0
- joint right_knee_joint: limit lower=0 upper=0 effort=0 velocity=0 -> lower=-2.792526803190927 upper=0 effort=0 velocity=0
- joint right_thigh_joint: limit lower=0 upper=0 effort=0 velocity=0 -> lower=-0.8726646259971648 upper=1.3089969389957472 effort=0 velocity=0
